Commit message: xacro correction

File: description/gazebo_control.xacro (robot description, xacro)
@@ -6,6 +6,6 @@
       <left_joint>left_wheel_joint</left_joint>
       <right_joint>right_wheel_joint</right_joint>
-      <wheel_separation>0.35</wheel_separation>
-      <wheel_diameter>0.1</wheel_diameter>
+      <wheel_separation>0.614</wheel_separation>
+      <wheel_diameter>0.25</wheel_diameter>
       <!-- Wheel Information -->
       <max_wheel_torque>200</max_wheel_torque>

File: description/robot_core.xacro (robot description, xacro)
@@ -18,5 +18,5 @@
   </link>
   <!-- Path to mesh -->
-  <xacro:property name="mesh_path" value="srs/my_bot/description/girello.stl" />
+  <xacro:property name="mesh_path" value="src/my_bot/description/girello.stl" />
   <!-- CHASSIS LINK -->
   <joint name="chassis_joint" type="fixed">
