Commit message: gazebo visual and control

File: description/robot_core.xacro (robot description, xacro)
@@ -41,4 +41,7 @@
     </xacro:inertial_box>
   </link>
+  <gazebo reference="chassis">
+    <material>Gazebo/White</material>
+  </gazebo>
   <!-- LEFT WHEEL LINK -->
   <joint name="left_wheel_joint" type="continuous">
@@ -64,4 +67,7 @@
     </xacro:inertial_cylinder>
   </link>
+  <gazebo reference="left_wheel">
+    <material>Gazebo/Blue</material>
+  </gazebo>
   <!-- RIGHT WHEEL LINK -->
   <joint name="right_wheel_joint" type="continuous">
@@ -87,4 +93,7 @@
     </xacro:inertial_cylinder>
   </link>
+  <gazebo reference="right_wheel">
+    <material>Gazebo/Blue</material>
+  </gazebo>
   <!-- CASTER WHEEL LINK -->
   <joint name="caster_wheel_joint" type="fixed">
@@ -110,3 +119,8 @@
     </xacro:inertial_sphere>
   </link>
+  <gazebo reference="caster_wheel">
+    <material>Gazebo/Black</material>
+    <mu1 value="0.001"/>
+    <mu2 value="0.001"/>
+  </gazebo>
 </robot>

Commit message: deambulator urdf visualization

File: description/robot_core.xacro (robot description, xacro)
@@ -17,4 +17,6 @@
   <link name="base_link">
   </link>
+  <!-- Path to mesh -->
+  <xacro:property name="mesh_path" value="mesh/girello.stl" />
   <!-- CHASSIS LINK -->
   <joint name="chassis_joint" type="fixed">
@@ -25,14 +27,16 @@
   <link name="chassis">
     <visual>
+      <origin xyz="0.1 0 0.075" rpy="${pi/2} 0 -${pi/2}"/>
+      <geometry>
+        <!--<box size="0.3 0.3 0.15"/>-->
+        <mesh filename="${mesh_path}" scale="0.01 0.01 0.01"/>
+      </geometry>
+      <material name="white"/>
+    </visual>
+    <collision>
       <origin xyz="0.15 0 0.075"/>
       <geometry>
         <box size="0.3 0.3 0.15"/>
-      </geometry>
-      <material name="white"/>
-    </visual>
-    <collision>
-      <origin xyz="0.15 0 0.075"/>
-      <geometry>
-        <box size="0.3 0.3 0.15"/>
+        <!--<mesh filename="${mesh_path}" scale="1 1 1"/>-->
       </geometry>
     </collision>
@@ -48,5 +52,5 @@
     <parent link="base_link"/>
     <child link="left_wheel"/>
-    <origin xyz="0 0.175 0" rpy="-${pi/2} 0 0"/>
+    <origin xyz="0 0.307 0" rpy="-${pi/2} 0 0"/>
     <axis xyz="0 0 1"/>
   </joint>
@@ -54,11 +58,11 @@
     <visual>
       <geometry>
-        <cylinder radius="0.05" length="0.04"/>
-      </geometry>
-      <material name="blue"/>
-    </visual>
-    <collision>
-      <geometry>
-        <cylinder radius="0.05" length="0.04"/>
+        <cylinder radius="0.125" length="0.04"/>
+      </geometry>
+      <material name="blue"/>
+    </visual>
+    <collision>
+      <geometry>
+        <cylinder radius="0.125" length="0.04"/>
       </geometry>
     </collision>
@@ -74,5 +78,5 @@
     <parent link="base_link"/>
     <child link="right_wheel"/>
-    <origin xyz="0 -0.175 0" rpy="${pi/2} 0 0"/>
+    <origin xyz="0 -0.307 0" rpy="${pi/2} 0 0"/>
     <axis xyz="0 0 -1"/>
   </joint>
@@ -80,11 +84,11 @@
     <visual>
       <geometry>
-        <cylinder radius="0.05" length="0.04"/>
-      </geometry>
-      <material name="blue"/>
-    </visual>
-    <collision>
-      <geometry>
-        <cylinder radius="0.05" length="0.04"/>
+        <cylinder radius="0.125" length="0.04"/>
+      </geometry>
+      <material name="blue"/>
+    </visual>
+    <collision>
+      <geometry>
+        <cylinder radius="0.125" length="0.04"/>
       </geometry>
     </collision>
@@ -96,31 +100,112 @@
     <material>Gazebo/Blue</material>
   </gazebo>
-  <!-- CASTER WHEEL LINK -->
-  <joint name="caster_wheel_joint" type="fixed">
+  <!-- LEFT FORK LINK -->
+  <joint name="left_fork_joint" type="continuous">
     <parent link="chassis"/>
-    <child link="caster_wheel"/>
-    <origin xyz="0.24 0 0"/>
-  </joint>
-  <link name="caster_wheel">
-    <visual>
-      <geometry>
-        <sphere radius="0.05"/>
-      </geometry>
-      <material name="black"/>
-    </visual>
-    <collision>
-      <geometry>
-        <sphere radius="0.05"/>
-      </geometry>
-      <material name="black"/>
-    </collision>
-    <xacro:inertial_sphere mass="0.1" radius="0.05">
-      <origin xyz="0 0 0" rpy="0 0 0"/>
-    </xacro:inertial_sphere>
-  </link>
-  <gazebo reference="caster_wheel">
+    <child link="left_fork"/>
+    <origin xyz="0.73 0.25 -0.03" rpy="0 0 0"/>
+    <axis xyz="0 0 1"/>
+  </joint>
+  <link name="left_fork">
+    <visual>
+      <geometry>
+        <cylinder radius="0.015" length="0.04"/>
+      </geometry>
+      <material name="blue"/>
+    </visual>
+    <collision>
+      <geometry>
+        <cylinder radius="0.015" length="0.04"/>
+      </geometry>
+    </collision>
+    <xacro:inertial_cylinder mass="0.1" length="0.04" radius="0.015">
+      <origin xyz="0 0 0" rpy="0 0 0"/>
+    </xacro:inertial_cylinder>
+  </link>
+  <gazebo reference="left_fork">
+    <material>Gazebo/Blue</material>
+  </gazebo>
+  <!-- LEFT CASTER WHEEL LINK -->
+    <joint name="left_cast_wheel_joint" type="continuous">
+    <parent link="left_fork"/>
+    <child link="left_caster_wheel"/>
+    <origin xyz="0.0 0.04 -0.0" rpy="${pi/2} 0 0"/>
+    <axis xyz="0 0 -1"/>
+  </joint>
+   <link name="left_caster_wheel">
+    <visual>
+      <geometry>
+        <cylinder radius="0.085" length="0.03"/>
+      </geometry>
+      <material name="blue"/>
+    </visual>
+    <collision>
+      <geometry>
+        <cylinder radius="0.085" length="0.03"/>
+      </geometry>
+    </collision>
+    <xacro:inertial_cylinder mass="0.1" length="0.03" radius="0.085">
+      <origin xyz="0 0 0" rpy="0 0 0"/>
+    </xacro:inertial_cylinder>
+  </link>
+  <gazebo reference="left_caster_wheel">
+    <material>Gazebo/Blue</material>
+  </gazebo>
+    <!-- RIGHT FORK LINK -->
+  <joint name="right_fork_joint" type="continuous">
+    <parent link="chassis"/>
+    <child link="right_fork"/>
+    <origin xyz="0.73 -0.25 -0.03" rpy="0 0 0"/>
+    <axis xyz="0 0 1"/>
+  </joint>
+  <link name="right_fork">
+        <visual>
+      <geometry>
+        <cylinder radius="0.015" length="0.04"/>
+      </geometry>
+      <material name="blue"/>
+    </visual>
+    <collision>
+      <geometry>
+        <cylinder radius="0.015" length="0.04"/>
+      </geometry>
+    </collision>
+    <xacro:inertial_cylinder mass="0.1" length="0.04" radius="0.015">
+      <origin xyz="0 0 0" rpy="0 0 0"/>
+    </xacro:inertial_cylinder>
+  </link>
+  <gazebo reference="right_fork">
+    <material>Gazebo/Blue</material>
+  </gazebo>
+  <!-- LEFT CASTER WHEEL LINK -->
+    <joint name="right_cast_wheel_joint" type="continuous">
+    <parent link="right_fork"/>
+    <child link="right_caster_wheel"/>
+    <origin xyz="0.0 -0.04 -0.0" rpy="${pi/2} 0 0"/>
+    <axis xyz="0 0 -1"/>
+  </joint>
+   <link name="right_caster_wheel">
+    <visual>
+      <geometry>
+        <cylinder radius="0.085" length="0.03"/>
+      </geometry>
+      <material name="blue"/>
+    </visual>
+    <collision>
+      <geometry>
+        <cylinder radius="0.085" length="0.03"/>
+      </geometry>
+    </collision>
+    <xacro:inertial_cylinder mass="0.1" length="0.03" radius="0.085">
+      <origin xyz="0 0 0" rpy="0 0 0"/>
+    </xacro:inertial_cylinder>
+  </link>
+  <gazebo reference="right_caster_wheel">
+    <material>Gazebo/Blue</material>
+  </gazebo>
+<!--   <gazebo reference="caster_wheel">
     <material>Gazebo/Black</material>
     <mu1 value="0.001"/>
     <mu2 value="0.001"/>
-  </gazebo>
+  </gazebo> -->
 </robot>

Commit message: corrected robot visualization

File: description/robot_core.xacro (robot description, xacro)
@@ -18,5 +18,5 @@
   </link>
   <!-- Path to mesh -->
-  <xacro:property name="mesh_path" value="mesh/girello.stl" />
+  <xacro:property name="mesh_path" value="srs/my_bot/description/girello.stl" />
   <!-- CHASSIS LINK -->
   <joint name="chassis_joint" type="fixed">
@@ -27,5 +27,5 @@
   <link name="chassis">
     <visual>
-      <origin xyz="0.1 0 0.075" rpy="${pi/2} 0 -${pi/2}"/>
+      <origin xyz="0.1 0 0.115" rpy="${pi/2} 0 -${pi/2}"/>
       <geometry>
         <!--<box size="0.3 0.3 0.15"/>-->
@@ -35,5 +35,5 @@
     </visual>
     <collision>
-      <origin xyz="0.15 0 0.075"/>
+      <origin xyz="0.15 0 0.115"/>
       <geometry>
         <box size="0.3 0.3 0.15"/>
@@ -41,6 +41,6 @@
       </geometry>
     </collision>
-    <xacro:inertial_box mass="0.5" x="0.3" y="0.3" z="0.15">
-      <origin xyz="0.15 0 0.075" rpy="0 0 0"/>
+    <xacro:inertial_box mass="0.5" x="0.5" y="0.7" z="0.15">
+      <origin xyz="0.15 0 0.115" rpy="0 0 0"/>
     </xacro:inertial_box>
   </link>
@@ -104,5 +104,5 @@
     <parent link="chassis"/>
     <child link="left_fork"/>
-    <origin xyz="0.73 0.25 -0.03" rpy="0 0 0"/>
+    <origin xyz="0.73 0.25 0.03" rpy="0 0 0"/>
     <axis xyz="0 0 1"/>
   </joint>
@@ -114,9 +114,9 @@
       <material name="blue"/>
     </visual>
-    <collision>
-      <geometry>
-        <cylinder radius="0.015" length="0.04"/>
-      </geometry>
-    </collision>
+<!--     <collision>
+      <geometry>
+        <cylinder radius="0.015" length="0.04"/>
+      </geometry>
+    </collision> -->
     <xacro:inertial_cylinder mass="0.1" length="0.04" radius="0.015">
       <origin xyz="0 0 0" rpy="0 0 0"/>
@@ -125,4 +125,6 @@
   <gazebo reference="left_fork">
     <material>Gazebo/Blue</material>
+    <mu1 value="0.01"/>
+    <mu2 value="0.01"/>
   </gazebo>
   <!-- LEFT CASTER WHEEL LINK -->
@@ -130,5 +132,5 @@
     <parent link="left_fork"/>
     <child link="left_caster_wheel"/>
-    <origin xyz="0.0 0.04 -0.0" rpy="${pi/2} 0 0"/>
+    <origin xyz="-0.04 0 -0.0875" rpy="${pi/2} 0 0"/>
     <axis xyz="0 0 -1"/>
   </joint>
@@ -136,14 +138,14 @@
     <visual>
       <geometry>
-        <cylinder radius="0.085" length="0.03"/>
-      </geometry>
-      <material name="blue"/>
-    </visual>
-    <collision>
-      <geometry>
-        <cylinder radius="0.085" length="0.03"/>
-      </geometry>
-    </collision>
-    <xacro:inertial_cylinder mass="0.1" length="0.03" radius="0.085">
+        <cylinder radius="0.0675" length="0.03"/>
+      </geometry>
+      <material name="blue"/>
+    </visual>
+    <collision>
+      <geometry>
+        <cylinder radius="0.0675" length="0.03"/>
+      </geometry>
+    </collision>
+    <xacro:inertial_cylinder mass="0.1" length="0.03" radius="0.0675">
       <origin xyz="0 0 0" rpy="0 0 0"/>
     </xacro:inertial_cylinder>
@@ -156,5 +158,5 @@
     <parent link="chassis"/>
     <child link="right_fork"/>
-    <origin xyz="0.73 -0.25 -0.03" rpy="0 0 0"/>
+    <origin xyz="0.73 -0.25 0.03" rpy="0 0 0"/>
     <axis xyz="0 0 1"/>
   </joint>
@@ -166,9 +168,9 @@
       <material name="blue"/>
     </visual>
-    <collision>
-      <geometry>
-        <cylinder radius="0.015" length="0.04"/>
-      </geometry>
-    </collision>
+<!--     <collision>
+      <geometry>
+        <cylinder radius="0.015" length="0.04"/>
+      </geometry>
+    </collision> -->
     <xacro:inertial_cylinder mass="0.1" length="0.04" radius="0.015">
       <origin xyz="0 0 0" rpy="0 0 0"/>
@@ -177,10 +179,12 @@
   <gazebo reference="right_fork">
     <material>Gazebo/Blue</material>
-  </gazebo>
-  <!-- LEFT CASTER WHEEL LINK -->
+    <mu1 value="0.01"/>
+    <mu2 value="0.01"/>
+  </gazebo>
+  <!-- RIGHT CASTER WHEEL LINK -->
     <joint name="right_cast_wheel_joint" type="continuous">
     <parent link="right_fork"/>
     <child link="right_caster_wheel"/>
-    <origin xyz="0.0 -0.04 -0.0" rpy="${pi/2} 0 0"/>
+    <origin xyz="-0.04 0 -0.0875" rpy="${pi/2} 0 0"/>
     <axis xyz="0 0 -1"/>
   </joint>
@@ -188,14 +192,14 @@
     <visual>
       <geometry>
-        <cylinder radius="0.085" length="0.03"/>
-      </geometry>
-      <material name="blue"/>
-    </visual>
-    <collision>
-      <geometry>
-        <cylinder radius="0.085" length="0.03"/>
-      </geometry>
-    </collision>
-    <xacro:inertial_cylinder mass="0.1" length="0.03" radius="0.085">
+        <cylinder radius="0.0675" length="0.03"/>
+      </geometry>
+      <material name="blue"/>
+    </visual>
+    <collision>
+      <geometry>
+        <cylinder radius="0.0675" length="0.03"/>
+      </geometry>
+    </collision>
+    <xacro:inertial_cylinder mass="0.1" length="0.03" radius="0.0675">
       <origin xyz="0 0 0" rpy="0 0 0"/>
     </xacro:inertial_cylinder>

Commit message: fixed visualization

File: description/robot_core.xacro (robot description, xacro)
@@ -18,5 +18,5 @@
   </link>
   <!-- Path to mesh -->
-  <xacro:property name="mesh_path" value="src/my_bot/description/girello.stl" />
+  <xacro:property name="mesh_path" value="srs/my_bot/description/girello.stl" />
   <!-- CHASSIS LINK -->
   <joint name="chassis_joint" type="fixed">

Commit message: fixed some things for presentation

File: description/robot_core.xacro (robot description, xacro)
@@ -35,8 +35,7 @@
     </visual>
     <collision>
-      <origin xyz="0.15 0 0.115"/>
-      <geometry>
-        <box size="0.3 0.3 0.15"/>
-        <!--<mesh filename="${mesh_path}" scale="1 1 1"/>-->
+      <origin xyz="0.4 0 0.115"/>
+      <geometry>
+        <box size="0.7 0.46 0.15"/>
       </geometry>
     </collision>

Commit message: visual update only when txt changes

File: description/robot_core.xacro (robot description, xacro)
@@ -18,5 +18,5 @@
   </link>
   <!-- Path to mesh -->
-  <xacro:property name="mesh_path" value="src/my_bot/description/girello.stl" />
+  <xacro:property name="mesh_path" value="srs/my_bot/description/girello.stl" />
   <!-- CHASSIS LINK -->
   <joint name="chassis_joint" type="fixed">
@@ -29,5 +29,4 @@
       <origin xyz="0.1 0 0.115" rpy="${pi/2} 0 -${pi/2}"/>
       <geometry>
-        <!--<box size="0.3 0.3 0.15"/>-->
         <mesh filename="${mesh_path}" scale="0.01 0.01 0.01"/>
       </geometry>
